File: Hardware/mcu.kicad_sch (KiCad schematic)
At the start: 44 parts, among them J101 DEBUG, SW101 Button_Left, SW102 Button_Middle, SW103 Button_Right, SW104 Boot_Select, SW105 RESET, U101 RP2040, U102 W25Q128JVPIQ TR, X101 12MHz

Commit message: Footprint Assignment
Parts:
- D101: footprint E61206RGBC3UDA:RGB_LED_E6C1206RGBC3UDA -> RamaPatchi:E6C1206RGBC3UDA
- D102: renamed from D202; footprint (none) -> RamaPatchi:HL-PC-3216S31YC-CZ
- J101: Package Size (none) -> 1206; Product Number (none) -> HL-PC-3216S31YC-CZ
- renumbered TP201 to TP101, TP201 to TP102
Changed lines of the file:
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@@
   (symbol (lib_id "RamaPotchi:LED") (at 284.48 221.615 180) (unit 1)
     (in_bom yes) (on_board yes) (dnp no)
-    (property "Reference" "D202" (at 284.48 224.155 0)
+    (property "Reference" "D102" (at 284.48 224.155 0)
       (effects (font (size 1.27 1.27)))
     )
@@
       (effects (font (size 1.27 1.27)) hide)
     )
-    (property "Footprint" "" (at 284.48 221.615 0)
+    (property "Footprint" "RamaPatchi:HL-PC-3216S31YC-CZ" (at 284.48 221.615 0)
       (effects (font (size 1.27 1.27)) hide)
     )
@@
     (instances
       (project "RamaPotchi"
-        (path "/d274aa36-eb9d-4efc-a7b7-51cc020ab33e/3d8c7fc1-a9db-40bc-9202-073c724f74f4"
-          (reference "D202") (unit 1)
-        )
         (path "/d274aa36-eb9d-4efc-a7b7-51cc020ab33e/2d8c086d-8126-4fa2-a232-1a618af9131f"
           (reference "D102") (unit 1)
@@
   (symbol (lib_id "RamaPotchi:TestPoint_Flag") (at 38.735 94.615 0) (mirror x) (unit 1)
     (in_bom yes) (on_board yes) (dnp no)
-    (property "Reference" "TP201" (at 39.37 99.06 0)
+    (property "Reference" "TP101" (at 39.37 99.06 0)
       (effects (font (size 1.27 1.27)) (justify left))
     )
@@
     (instances
       (project "RamaPotchi"
-        (path "/d274aa36-eb9d-4efc-a7b7-51cc020ab33e/3d8c7fc1-a9db-40bc-9202-073c724f74f4"
-          (reference "TP201") (unit 1)
-        )
         (path "/d274aa36-eb9d-4efc-a7b7-51cc020ab33e/2d8c086d-8126-4fa2-a232-1a618af9131f"
           (reference "TP101") (unit 1)
@@
       (effects (font (size 1.27 1.27)))
     )
-    (property "Footprint" "E61206RGBC3UDA:RGB_LED_E6C1206RGBC3UDA" (at 378.46 159.385 0)
-      (effects (font (size 1.27 1.27)) hide)
-    )
-    (property "Datasheet" "~" (at 378.46 159.385 0)
+    (property "Footprint" "RamaPatchi:E6C1206RGBC3UDA" (at 378.46 159.385 0)
+      (effects (font (size 1.27 1.27)) hide)
+    )
+    (property "Datasheet" "https://datasheet.lcsc.com/lcsc/2203301730_EKINGLUX-E6C1206RGBC3UDA_C375571.pdf" (at 378.46 159.385 0)
       (effects (font (size 1.27 1.27)) hide)
     )
@@
       (effects (font (size 1.27 1.27)) hide)
     )
-    (property "Datasheet" "~" (at 215.265 217.805 0)
-      (effects (font (size 1.27 1.27)) hide)
+    (property "Datasheet" "https://datasheet.lcsc.com/lcsc/2307111134_HCTL-XH-3A-P_C2979572.pdf" (at 215.265 217.805 0)
+      (effects (font (size 1.27 1.27)) hide)
+    )
+    (property "Package Size" "1206" (at 215.265 217.805 0)
+      (effects (font (size 1.27 1.27)) hide)
+    )
+    (property "Product Number" "HL-PC-3216S31YC-CZ" (at 218.44 224.79 0)
+      (effects (font (size 1.27 1.27)))
     )
     (pin "3")
@@
   (symbol (lib_id "RamaPotchi:TestPoint_Flag") (at 126.365 208.28 0) (mirror x) (unit 1)
     (in_bom yes) (on_board yes) (dnp no)
-    (property "Reference" "TP201" (at 127 212.725 0)
+    (property "Reference" "TP102" (at 127 212.725 0)
       (effects (font (size 1.27 1.27)) (justify left))
     )
@@
     (instances
       (project "RamaPotchi"
-        (path "/d274aa36-eb9d-4efc-a7b7-51cc020ab33e/3d8c7fc1-a9db-40bc-9202-073c724f74f4"
-          (reference "TP201") (unit 1)
-        )
         (path "/d274aa36-eb9d-4efc-a7b7-51cc020ab33e/2d8c086d-8126-4fa2-a232-1a618af9131f"
           (reference "TP102") (unit 1)
