File: Hardware/power_battery_data.kicad_sch (KiCad schematic)
At the start: 32 parts, among them J201 USB_C_Receptacle_USB2.0, Q201 FS8205A, Q202 DMG2305UX-13, U201 TP4056, U202 DW01A, U204 RT6150B-33GQW

Commit message: Footprint Assignment
Parts:
- CR201: footprint MBR120VLSFT1G:SDO_SOD-123FL_ONS -> RamaPatchi:SDO_SOD-123FL_ONS
- D201: footprint (none) -> RamaPatchi:HL-PC-3261S9AC; Package Size (none) -> 1206; Part Number (none) -> HL-PC-3216S9AC
- D202: footprint (none) -> RamaPatchi:HL-PC-3216U51GC; Package Size (none) -> 1206; Part Number (none) -> HL-PC-3216U51GC
- renumbered R112 to R201, R113 to R202
Changed lines of the file:
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@@
       (effects (font (size 1.524 1.524)))
     )
-    (property "Footprint" "MBR120VLSFT1G:SDO_SOD-123FL_ONS" (at 278.765 185.42 0)
+    (property "Footprint" "RamaPatchi:SDO_SOD-123FL_ONS" (at 278.765 185.42 0)
       (effects (font (size 1.27 1.27) italic) hide)
     )
@@
   (symbol (lib_id "RamaPotchi:R") (at 93.345 67.945 90) (unit 1)
     (in_bom yes) (on_board yes) (dnp no)
-    (property "Reference" "R113" (at 93.345 70.485 90)
+    (property "Reference" "R202" (at 93.345 70.485 90)
       (effects (font (size 1.27 1.27)))
     )
@@
     (instances
       (project "RamaPotchi"
-        (path "/d274aa36-eb9d-4efc-a7b7-51cc020ab33e/2d8c086d-8126-4fa2-a232-1a618af9131f"
-          (reference "R113") (unit 1)
-        )
         (path "/d274aa36-eb9d-4efc-a7b7-51cc020ab33e/3d8c7fc1-a9db-40bc-9202-073c724f74f4"
           (reference "R202") (unit 1)
@@
       (effects (font (size 1.27 1.27)) hide)
     )
-    (property "Footprint" "" (at 53.34 165.1 0)
-      (effects (font (size 1.27 1.27)) hide)
-    )
-    (property "Datasheet" "~" (at 53.34 165.1 0)
+    (property "Footprint" "RamaPatchi:HL-PC-3261S9AC" (at 53.34 165.1 0)
+      (effects (font (size 1.27 1.27)) hide)
+    )
+    (property "Datasheet" "https://datasheet.lcsc.com/lcsc/2009091206_HONGLITRONIC-Hongli-Zhihui--HONGLITRONIC-HL-PC-3216S9AC_C499470.pdf" (at 53.34 165.1 0)
       (effects (font (size 1.27 1.27)) hide)
     )
@@
       (effects (font (size 1.27 1.27)))
     )
+    (property "Part Number" "HL-PC-3216S9AC" (at 55.88 173.99 0)
+      (effects (font (size 1.27 1.27)))
+    )
+    (property "Package Size" "1206" (at 53.34 165.1 0)
+      (effects (font (size 1.27 1.27)) hide)
+    )
     (pin "1")
     (pin "2")
@@
   (symbol (lib_id "RamaPotchi:R") (at 93.345 62.865 90) (unit 1)
     (in_bom yes) (on_board yes) (dnp no)
-    (property "Reference" "R112" (at 93.345 58.42 90)
+    (property "Reference" "R201" (at 93.345 58.42 90)
       (effects (font (size 1.27 1.27)))
     )
@@
     (instances
       (project "RamaPotchi"
-        (path "/d274aa36-eb9d-4efc-a7b7-51cc020ab33e/2d8c086d-8126-4fa2-a232-1a618af9131f"
-          (reference "R112") (unit 1)
-        )
         (path "/d274aa36-eb9d-4efc-a7b7-51cc020ab33e/3d8c7fc1-a9db-40bc-9202-073c724f74f4"
           (reference "R201") (unit 1)
@@
       (effects (font (size 1.27 1.27)) hide)
     )
-    (property "Footprint" "" (at 53.34 178.435 0)
-      (effects (font (size 1.27 1.27)) hide)
-    )
-    (property "Datasheet" "~" (at 53.34 178.435 0)
+    (property "Footprint" "RamaPatchi:HL-PC-3216U51GC" (at 53.34 178.435 0)
+      (effects (font (size 1.27 1.27)) hide)
+    )
+    (property "Datasheet" "https://datasheet.lcsc.com/lcsc/2009091206_HONGLITRONIC-Hongli-Zhihui--HONGLITRONIC-HL-PC-3216U51GC_C499467.pdf" (at 53.34 178.435 0)
       (effects (font (size 1.27 1.27)) hide)
     )
@@
       (effects (font (size 1.27 1.27)))
     )
+    (property "Package Size" "1206" (at 53.34 178.435 0)
+      (effects (font (size 1.27 1.27)) hide)
+    )
+    (property "Part Number" "HL-PC-3216U51GC" (at 53.34 186.69 0)
+      (effects (font (size 1.27 1.27)))
+    )
